File: esp_car.brd (EAGLE design)
At the start: 160 x 100 mm, 12 parts, among them IC1 TB6612FNG, U1 ESP-WROOM-32

Commit message: daliy commit
Parts:
- added 5VOUT: (no value), jst-xh:S2B-XH-A
- added C6: 10uF, rcl:C1608
- added EN(RESET), IO0（BOOT): P-06185_SKRPACE010, Akizuki:SKRP
- added ML, MR: B6B-ZR, jst:B6B-ZR
- moved NDS9936 74.4 mm to (30.5, 44.5), turned to 90 degrees
- moved U1 45.8 mm to (22.9, 17.8)
- moved JP1 45.7 mm to (10.2, 43.2)
Connections:
- removed net N$1: NDS9936.7, NDS9936.8
- removed net N$2: NDS9936.5, NDS9936.6
- removed net N$3: NDS9936.1, NDS9936.4
- removed net N$4: NDS9936.2, NDS9936.3
- removed net N$5: C5.2, R1.1
- new net DTR: JP1.6, NDS9936.2, NDS9936.3
- new net EN: C5.2, EN(RESET).2A, NDS9936.7, NDS9936.8, R1.1, U1.3
- new net IO0: IO0（BOOT).1A, NDS9936.5, NDS9936.6, U1.25
- new net RTS: JP1.2, NDS9936.1, NDS9936.4
- new net RX: JP1.4, U1.34
- new net TX: JP1.5, U1.35
- net +3V3: now also C6.2, JP1.3
- net +5V: now also 5VOUT.2
- net GND: now also 5VOUT.1, C6.1, EN(RESET).1A, IO0（BOOT).2A, JP1.1

Commit message: daliy commit
Parts:
- added C8: 100u, rcl:E2,5-6
- added SW2: SK-12D01, Seeed-OPL-Button:SW5-2.0-8.8X4.4X4.7MM-90D
- added U$5, U$7: 2.0, Mount_pad:2.0
Connections:
- net GND: now also C8.-, U$5.P$1
- net VCC: now also C2.1, C3.1, NJM2391.1, NJM7805.1, SW2.COM
- net VDD: now also C8.+, SW2.A, U$7.P$1; no longer C2.1, C3.1, NJM2391.1, NJM7805.1
Changed lines of the file:
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@@
 <attribute name="SPICEPREFIX" value="C" x="-66.04" y="-43.18" size="1.778" layer="27" display="off"/>
+</element>
+<element name="C8" library="rcl" package="E2,5-6" value="100u" x="-58.42" y="-137.16"/>
+<element name="U$5" library="Mount_pad" package="2.0" value="2.0" x="-53.34" y="-81.28"/>
+<element name="U$7" library="Mount_pad" package="2.0" value="2.0" x="-53.34" y="-111.76"/>
+<element name="SW2" library="Seeed-OPL-Button" package="SW5-2.0-8.8X4.4X4.7MM-90D" value="SK-12D01" x="-78.74" y="-132.08">
+<attribute name="MPN" value="SK-12D01" x="-78.74" y="-132.08" size="1.778" layer="27" display="off"/>
 </element>
 </elements>
@@
 <contactref element="U1" pad="GND"/>
 <contactref element="C6" pad="1"/>
+<contactref element="C8" pad="-"/>
+<contactref element="U$5" pad="P$1"/>
+<wire x1="-53.34" y1="-81.28" x2="-57.15" y2="-137.16" width="0" layer="19" extent="1-1"/>
+<wire x1="-66.89" y1="-43.18" x2="-53.34" y2="-81.28" width="0" layer="19" extent="1-1"/>
 <wire x1="-59.71" y1="-30.48" x2="-66.89" y2="-43.18" width="0" layer="19" extent="1-1"/>
 <wire x1="-48.075" y1="-10.925" x2="-59.71" y2="-30.48" width="0" layer="19" extent="1-1"/>
@@
 <signal name="VCC">
 <contactref element="IC1" pad="20"/>
+<contactref element="C2" pad="1"/>
+<contactref element="NJM2391" pad="1"/>
+<contactref element="NJM7805" pad="1"/>
+<contactref element="C3" pad="1"/>
+<contactref element="SW2" pad="COM"/>
+<wire x1="-41.65" y1="1.55" x2="-78.74" y2="-132.08" width="0" layer="19" extent="1-1"/>
+<wire x1="-21.33" y1="30.76" x2="-41.65" y2="1.55" width="0" layer="19" extent="1-1"/>
+<wire x1="-33.995" y1="37.915" x2="-21.33" y2="30.76" width="0" layer="19" extent="1-1"/>
+<wire x1="-49.11" y1="44.45" x2="-33.995" y2="37.915" width="0" layer="19" extent="1-1"/>
+<wire x1="-18.63" y1="49.53" x2="-21.33" y2="30.76" width="0" layer="19" extent="1-1"/>
 </signal>
 <signal name="VM1">
@@
 </signal>
 <signal name="VDD">
-<contactref element="C2" pad="1"/>
-<contactref element="NJM2391" pad="1"/>
-<contactref element="NJM7805" pad="1"/>
-<contactref element="C3" pad="1"/>
+<contactref element="C8" pad="+"/>
+<contactref element="U$7" pad="P$1"/>
+<contactref element="SW2" pad="A"/>
+<wire x1="-59.69" y1="-137.16" x2="-78.74" y2="-130.048" width="0" layer="19" extent="1-1"/>
+<wire x1="-53.34" y1="-111.76" x2="-59.69" y2="-137.16" width="0" layer="19" extent="1-1"/>
 </signal>
 <signal name="+3V3">

Commit message: chematic v1.0
Parts:
- removed NJM2391: 7806DT, linear:TO252
- removed U1: ESP-WROOM-32, esp32 (2):ESP-WROOM-32
- added C10, C9: 0.1u, rcl:C1608
- added C11, C12, C13: 0.1uF, rcl:C1608
- added GY-530C, GY-530L, GY-530R: (no value), pinhead:1X05M
- added GY-91: (no value), adafruit:1X06
- added IC2: LT1963ES8-3.3, linear-technology:SOIC8
- added JP4: (no value), pinhead:1X10
- added LED5, LED6, LED7, LED8: WS2812B5050, adafruit:WS2812B
- added R2: 10k, rcl:R0603
- added R3: 4.7k, rcl:R0603
- added R4: 4.7K, rcl:R0603
- added SJ1: (no value), SparkFun:SJ_3
- added T0, T1, T2, T3, T5, T7: (no value), wirepad:SMD2,54-5,08
- added U$6: PB04, Buzzer:PB04
- added U2: ESP-WROOM-32_NOFLASH, esp32 _my:ESP-WROOM-32_NOFLASH
- C2, C3: value 0.1uF -> 10uF
- moved U$7 188.0 mm to (-49.5, 76.2)
- moved C8 186.7 mm to (-59.7, 49.5)
- moved U$5 157.7 mm to (-45.7, 76.2)
- moved SW2 143.3 mm to (-47.0, 7.62)
- moved C6 113.0 mm to (-66.0, 69.8)
- moved ML 85.4 mm to (-38.1, 52.1)
- moved NDS9936 84.4 mm to (-53.3, 34.3), turned to 0 degrees
- moved IO0（BOOT) 75.6 mm to (-43.2, 63.5)
- moved MR 72.6 mm to (-50.8, 52.1)
- moved EN(RESET) 70.9 mm to (-31.8, 63.5)
- moved JP1 41.5 mm to (-21.6, 69.8)
- moved 5VOUT 33.2 mm to (-57.1, 2.54)
- moved C1 30.6 mm to (-53.3, 69.8)
- moved C5 30.6 mm to (-47.0, 69.8)
- moved C3 30.6 mm to (-40.6, 69.8)
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Connections:
- removed net PGND1: IC1.3
- removed net PGND1': IC1.4
- removed net PGND2: IC1.9
- removed net PGND2': IC1.10
- removed net VM1: IC1.24
- removed net VM2: IC1.13
- removed net VM3: IC1.14
- new net ENCL_A: ML.3, U2.6
- new net ENCL_B: ML.4, U2.7
- new net ENCR_A: MR.3, U2.4
- new net ENCR_B: MR.4, U2.5
- new net I2C_SCL: GY-530C.3, GY-530L.3, GY-530R.3, GY-91.3, JP4.4, R3.1, U2.36
- new net I2C_SDA: GY-530C.4, GY-530L.4, GY-530R.4, GY-91.4, JP4.5, R4.1, U2.33
- new net IO12: JP4.9, T5.1, U2.14
- new net IO15: JP4.8, T3.1, U2.23
- new net IO2: JP4.6, T2.1, U2.24
- new net IO27: JP4.10, T7.1, U2.12
- new net IO4: T0.1, U2.26
- new net IO5: JP4.7, U2.29
- new net ML_IN1: IC1.21, U2.27
- new net ML_IN2: IC1.22, U2.28
- new net ML_PWM: IC1.23, U2.11
- new net MR_IN1: IC1.17, U2.30
- new net MR_IN2: IC1.16, U2.31
- new net MR_PWM: IC1.15, U2.10
- new net N$10: IC1.1, IC1.2, ML.1
- new net N$11: IC1.5, IC1.6, ML.6
- new net N$12: IC1.7, IC1.8, MR.6
- new net N$13: IC1.11, IC1.12, MR.1
- new net N$15: LED7.2-DOUT, LED8.4-DIN
- new net N$18: LED5.4-DIN, U2.16
- new net N$19: GY-530R.5, U2.9
- new net N$2: IC2.8
- new net N$3: GY-530L.5, U2.8
- new net N$4: GY-91.6, SJ1.2
- new net N$5: GY-530C.5, U2.37
- new net N$6: LED5.2-DOUT, LED6.4-DIN
- new net N$7: IC1.19, R2.1
- new net N$8: U$6.P$1, U2.13
- new net N$9: LED6.2-DOUT, LED7.4-DIN
- net +3V3: now also C9.1, GY-530C.1, GY-530L.1, GY-530R.1, GY-91.1, GY-91.5, IC1.20, IC2.1, IC2.2, JP4.3, ML.2, MR.2, R2.2, R4.2, SJ1.3, U2.2; no longer NJM2391.2, U1.2
- net +5V: now also C11.1, C12.1, C13.1, JP4.2, LED5.1-VDD, LED6.1-VDD, LED7.1-VDD, LED8.1-VDD
- net EN: now also U2.3; no longer U1.3
- net GND: now also C10.2, C11.2, C12.2, C13.2, C9.2, GY-530C.2, GY-530L.2, GY-530R.2, GY-91.2, IC1.10, IC1.3, IC1.4, IC1.9, IC2.3, IC2.6, IC2.7, JP4.1, LED5.3-GND, LED6.3-GND, LED7.3-GND, LED8.3-GND, ML.5, MR.5, SJ1.1, U$6.P$2, U2.1, U2.15, U2.38, U2.GND; no longer NJM2391.3, U1.1, U1.15, U1.38, U1.GND
- net IO0: now also T1.1, U2.25; no longer U1.25
- net RX: now also U2.34; no longer U1.34
- net TX: now also U2.35; no longer U1.35
- net VCC: now also IC2.5; no longer IC1.20, NJM2391.1
- net VDD: now also C10.1, IC1.13, IC1.14, IC1.24
Other:
- board size 160 x 100 mm -> 168 x 168 mm

Commit message: board test
Parts:
- removed JP1: (no value), adafruit:1X06
- removed JP4: (no value), pinhead:1X10
- added SERIAL: (no value), adafruit:1X06
- added UNIV: (no value), pinhead:1X10
- moved IC2 224.0 mm to (70.6, 55.6), turned to 90 degrees
- moved GY-530R 156.5 mm to (67.6, 68.3), turned to 135 degrees
- moved T3 145.5 mm to (-15.2, 66.0)
- moved T7 143.4 mm to (-25.4, 66.0)
- moved C13 134.0 mm to (-36.8, 77.5)
- moved C12 130.7 mm to (-30.5, 77.5)
- moved C11 127.7 mm to (-24.1, 77.5)
- moved T2 124.5 mm to (-72.4, 58.4)
- moved MR 114.1 mm to (61.2, 30.5), turned to 180 degrees
- moved GY-530L 105.7 mm to (11.9, 68.3), turned to 225 degrees
- moved GY-530C 96.7 mm to (40.6, 80.0)
- moved LED5 96.1 mm to (66.0, 11.4), turned to 45 degrees
- moved GY-91 95.4 mm to (39.4, 47.0)
- moved IO0（BOOT) 94.1 mm to (50.3, 74.7), turned to 90 degrees
- moved 5VOUT 94.0 mm to (36.8, 1.27), turned to 350 degrees
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Connections:
- net +3V3: now also SERIAL.3, UNIV.3; no longer JP1.3, JP4.3
- net +5V: now also UNIV.2; no longer JP4.2
- net DTR: now also SERIAL.6; no longer JP1.6
- net GND: now also SERIAL.1, UNIV.1; no longer JP1.1, JP4.1
- net I2C_SCL: now also UNIV.4; no longer JP4.4
- net I2C_SDA: now also UNIV.5; no longer JP4.5
- net IO12: now also UNIV.9; no longer JP4.9
- net IO15: now also UNIV.8; no longer JP4.8
- net IO2: now also UNIV.6; no longer JP4.6
- net IO27: now also UNIV.10; no longer JP4.10
- net IO5: now also UNIV.7; no longer JP4.7
- net RTS: now also SERIAL.2; no longer JP1.2
- net RX: now also SERIAL.4; no longer JP1.4
- net TX: now also SERIAL.5; no longer JP1.5
Other:
- board size 168 x 168 mm -> 90 x 84 mm

Commit message: sche fix,board test
Parts:
- removed T7: (no value), wirepad:SMD2,54-5,08
- removed U$6: PB04, Buzzer:PB04
- added BUZ+, BUZ-: (no value), wirepad:SMD1,27-2,54
- added R5: 10k, rcl:R0603
- added R6: 20k, rcl:R0603
- 5VOUT: device jst-xh:S2B-XH-A -> jst-xh:B2B-XH-A
- UNIV: device pinhead:1X10 -> adafruit:1X09-BIG
- moved T0 135.8 mm to (69.8, 17.4), flipped to the bottom
- moved T1 130.4 mm to (55.2, 7.42), flipped to the bottom
- moved T2 110.0 mm to (25.1, 7.42), flipped to the bottom
- moved UNIV 105.1 mm to (-12.0, 2.00), turned to 90 degrees
- moved LED6 76.6 mm to (13.9, 11.7)
- moved LED7 76.0 mm to (58.0, 73.4)
- moved T5 74.5 mm to (40.2, 22.5), flipped to the bottom
- moved IC2 59.0 mm to (11.6, 56.6)
- moved T3 54.6 mm to (9.76, 17.5), flipped to the bottom
- moved NJM7805 47.3 mm to (65.0, 59.6)
- moved 5VOUT 41.0 mm to (71.0, 24.0), turned to 0 degrees
- moved ML 35.3 mm to (54.1, 50.0)
- moved MR 35.0 mm to (26.2, 30.0)
- moved IC1 34.2 mm to (56.2, 59.9), turned to 90 degrees
- moved C8 19.0 mm to (18.1, 49.5), turned to 180 degrees
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Connections:
- net +5V: now also 5VOUT.1; no longer 5VOUT.2
- net GND: now also 5VOUT.2, BUZ-.1, R5.1; no longer 5VOUT.1, U$6.P$2
- net IO27: now also R5.2, R6.1; no longer T7.1, UNIV.10
- net N$8: now also BUZ+.1; no longer U$6.P$1
- net VDD: now also R6.2
Other:
- board size 90 x 84 mm -> 81.6 x 84 mm

Commit message: pdf add
Parts:
- added C14: 0.1uF, rcl:C1608
- moved C4 122.0 mm to (49.2, 27.8), turned to 180 degrees
- moved C3 114.5 mm to (49.0, 31.6), turned to 180 degrees
- moved SJ1 108.6 mm to (50.2, 48.7), turned to 90 degrees
- moved C6 96.1 mm to (26.9, 67.0)
- moved R5 92.0 mm to (27.5, 53.5), turned to 180 degrees
- moved R2 91.3 mm to (30.9, 27.4), turned to 180 degrees
- moved R6 91.3 mm to (27.5, 49.0), turned to 180 degrees
- moved R3 86.8 mm to (53.8, 67.5)
- moved R4 76.0 mm to (58.0, 67.5)
- moved C10 75.6 mm to (28.4, 30.8), turned to 90 degrees
- moved C9 75.5 mm to (33.5, 30.9), turned to 90 degrees
- moved R1 68.5 mm to (27.2, 58.0)
- moved C1 67.8 mm to (23.0, 62.8), turned to 90 degrees
- moved C2 62.4 mm to (10.0, 59.0), turned to 90 degrees
- moved C5 47.3 mm to (27.2, 63.0)
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Connections:
- net +5V: now also C14.1
- net GND: now also C14.2
Routing:
- net GND: track 0.00 -> 479.3 mm, vias 0 -> 2
- net +5V: track 0.00 -> 275.9 mm, vias 0 -> 3
- net +3V3: track 0.00 -> 228.9 mm, vias 0 -> 5
- net VCC: track 0.00 -> 135.9 mm, vias 0 -> 1
- net I2C_SCL: track 0.00 -> 116.7 mm, vias 0 -> 3
- net I2C_SDA: track 0.00 -> 114.4 mm, vias 0 -> 4
- net N$9: track 0.00 -> 104.3 mm, vias 0 -> 2
- net VDD: track 0.00 -> 96.6 mm, vias 0 -> 3
- net IO15: track 0.00 -> 92.2 mm, vias 0 -> 1
- net MR_PWM: track 0.00 -> 88.5 mm
- net IO0: track 0.00 -> 70.1 mm, vias 0 -> 2
- net N$6: track 0.00 -> 68.6 mm
- net N$18: track 0.00 -> 65.0 mm, vias 0 -> 2
- net IO12: track 0.00 -> 62.7 mm, vias 0 -> 1
- net ENCR_A: track 0.00 -> 58.2 mm, vias 0 -> 3
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
Commit message: from office
Parts:
- 5VOUT: device jst-xh:B2B-XH-A -> pinhead:1X02
- moved C14 112.7 mm to (72.0, 22.0)
- moved UNIV 108.3 mm to (62.5, 54.5), turned to 180 degrees
- moved C12 83.0 mm to (52.5, 77.5)
- moved C13 72.2 mm to (11.2, 23.5)
- moved C11 52.0 mm to (27.9, 76.5)
- moved NDS9936 42.5 mm to (16.1, 57.5), turned to 180 degrees
- moved SERIAL 36.6 mm to (23.4, 61.5), turned to 90 degrees
- moved IO0（BOOT) 24.7 mm to (27.0, 67.0)
- moved C8 22.4 mm to (28.1, 29.5)
- moved C3 22.0 mm to (71.0, 31.6)
- moved C4 22.0 mm to (71.2, 27.8)
- moved MR 20.8 mm to (20.8, 50.0), turned to 0 degrees
- moved R3 16.1 mm to (52.0, 51.5)
- moved R4 16.0 mm to (57.0, 51.5)
- moved U$5 15.9 mm to (22.0, 31.9)
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Routing:
- net GND: track 479.3 -> 385.3 mm, vias 2 -> 8
- net I2C_SDA: track 114.4 -> 190.6 mm, vias 4 -> 3
- net MR_IN2: track 38.2 -> 95.8 mm
- net IO0: track 70.1 -> 126.0 mm, vias 2 -> 10
- net MR_PWM: track 88.5 -> 39.9 mm, vias 0 -> 2
- net +5V: track 275.9 -> 235.3 mm, vias 3 -> 5
- net ML_IN1: track 32.7 -> 70.9 mm, vias 2 -> 4
- net ML_PWM: track 36.0 -> 0.00 mm, vias 2 -> 0
- net ENCR_B: track 57.7 -> 23.7 mm, vias 2 -> 0
- net ENCR_A: track 58.2 -> 25.8 mm
- net IO4: track 50.9 -> 78.4 mm, vias 1 -> 3
- net IO2: track 53.4 -> 79.2 mm, vias 3 -> 8
- net N$9: track 104.3 -> 80.6 mm, vias 2 -> 4
- net VDD: track 96.6 -> 74.1 mm, vias 3 -> 1
- net ML_IN2: track 33.1 -> 55.5 mm, vias 2 -> 6
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
Commit message: daily
Parts:
- removed LED5, LED6, LED7, LED8: WS2812B5050, adafruit:WS2812B
- added LED_FL, LED_FR, LED_RL, LED_RR: WS2812B5050, adafruit:WS2812B
- GY-530C, GY-530L, GY-530R: device pinhead:1X05M -> pinhead:1X05
- moved C12 69.1 mm to (12.0, 21.5), turned to 180 degrees
- moved C13 62.3 mm to (73.3, 19.5), turned to 180 degrees
- moved C14 57.9 mm to (51.0, 76.0), turned to 270 degrees
- moved C9 40.8 mm to (41.0, 68.0), turned to 270 degrees
- moved R2 39.0 mm to (38.0, 68.0), turned to 180 degrees
- moved C10 37.3 mm to (44.0, 68.0), turned to 90 degrees
- moved MR 36.3 mm to (57.0, 47.0), turned to 180 degrees
- moved IC1 28.3 mm to (40.5, 58.5), turned to 0 degrees
- moved R3 23.4 mm to (47.0, 74.5), turned to 180 degrees
- moved R4 23.2 mm to (45.0, 71.5), turned to 180 degrees
- moved SJ1 17.5 mm to (34.9, 27.6), turned to 0 degrees
- moved ML 16.4 mm to (33.0, 47.0), turned to 180 degrees
- moved GY-91 15.5 mm to (40.0, 32.5)
- moved BUZ+ 15.4 mm to (25.0, 54.0), turned to 0 degrees
- moved R6 11.7 mm to (34.5, 54.0), turned to 270 degrees
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- renumbered U2 to U1
Connections:
- net N$10 renamed ML+
- net N$11 renamed ML-
- net N$12 renamed MR-
- net N$13 renamed MR+
- removed net N$2: IC2.8
- net +3V3: now also R3.2
- net +5V: now also LED_FL.1-VDD, LED_FR.1-VDD, LED_RL.1-VDD, LED_RR.1-VDD; no longer LED5.1-VDD, LED6.1-VDD, LED7.1-VDD, LED8.1-VDD
- net GND: now also LED_FL.3-GND, LED_FR.3-GND, LED_RL.3-GND, LED_RR.3-GND; no longer LED5.3-GND, LED6.3-GND, LED7.3-GND, LED8.3-GND, U1.GND
- net N$15: now also LED_FR.4-DIN, LED_RR.2-DOUT; no longer LED7.2-DOUT, LED8.4-DIN
- net N$18: now also LED_FL.4-DIN; no longer LED5.4-DIN
- net N$19: now also GY-530L.5; no longer GY-530R.5
- net N$3: now also GY-530C.5; no longer GY-530L.5
- net N$5: now also GY-530R.5; no longer GY-530C.5
- net N$6: now also LED_FL.2-DOUT, LED_RL.4-DIN; no longer LED5.2-DOUT, LED6.4-DIN
- net N$9: now also LED_RL.2-DOUT, LED_RR.4-DIN; no longer LED6.2-DOUT, LED7.4-DIN
- net VCC: now also IC2.8
Routing:
- net GND: track 385.3 -> 0.00 mm, vias 8 -> 0
- net +5V: track 235.3 -> 0.00 mm, vias 5 -> 0
- net +3V3: track 217.0 -> 0.00 mm, vias 10 -> 0
- net I2C_SDA: track 190.6 -> 0.00 mm, vias 3 -> 0
- net I2C_SCL: track 129.1 -> 0.00 mm, vias 3 -> 0
- net VCC: track 128.0 -> 0.00 mm, vias 4 -> 0
- net IO0: track 126.0 -> 0.00 mm, vias 10 -> 0
- net MR_IN2: track 95.8 -> 0.00 mm, vias 4 -> 0
- net N$9: track 80.6 -> 0.00 mm, vias 4 -> 0
- net IO2: track 79.2 -> 0.00 mm, vias 8 -> 0
- net IO4: track 78.4 -> 0.00 mm, vias 3 -> 0
- net IO12: track 76.1 -> 0.00 mm, vias 8 -> 0
- net VDD: track 74.1 -> 0.00 mm, vias 1 -> 0
- net ML_IN1: track 70.9 -> 0.00 mm, vias 4 -> 0
- net IO15: track 69.8 -> 0.00 mm, vias 6 -> 0
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Other:
- outline, holes or cut-outs redrawn
