File: esp_car.sch (EAGLE design)
At the start: 12 parts, among them IC1 TB6612FNG, U1 ESP-WROOM-32

Commit message: daliy commit
Parts:
- added 5VOUT: (no value), jst-xh:S2B-XH-A
- added C6: 10uF, rcl:C-EUC1608
- added EN(RESET), IO0（BOOT): P-06185_SKRPACE010, Akizuki:P-06185_SKRPACE010
- added ML, MR: B6B-ZR, jst:B6B-ZR
Connections:
- removed net N$1: NDS9936A.D
- removed net N$2: NDS9936B.D
- removed net N$3: NDS9936A.S, NDS9936B.G
- removed net N$4: NDS9936A.G, NDS9936B.S
- removed net N$5: C5.2, R1.1
- new net DTR: JP1.6, NDS9936A.G, NDS9936B.S
- new net EN: C5.2, EN(RESET).P$2A, NDS9936A.D, R1.1, U1.EN
- new net IO0: IO0（BOOT).P$1A, NDS9936B.D, U1.IO0
- new net RTS: JP1.2, NDS9936A.S, NDS9936B.G
- new net RX: JP1.4, U1.RXD0
- new net TX: JP1.5, U1.TXD0
- net +3V3: now also C6.2, JP1.3
- net +5V: now also 5VOUT.2
- net GND: now also 5VOUT.1, C6.1, EN(RESET).P$1A, IO0（BOOT).P$2A, JP1.1, U1.GND@1, U1.GND@2, U1.GND@3, U1.GND@4
Other:
- note added: "DTR RX TX VCC RTS GND"
- note removed: "DTR"
- note removed: "EN"
- note removed: "IO0"
- note removed: "RTS"
- moved on the sheet: C5, IC1, JP1, R1, U1

Commit message: daliy commit
Parts:
- added C8: 100u, rcl:CPOL-USE2.5-6
- added SW2: SK-12D01, Seeed-OPL-Button:DIP-TOGGLE-SWITCH-ON-ON(3+2P-8.8X4.6MM)
- added U$5, U$7: 2.0, Mount_pad:2.0
Connections:
- new net VCC: C2.1, C3.1, NJM2391.VI, NJM7805.VI, SW2.COM
- net GND: now also C8.-, U$5.P$1
- net VDD: now also C8.+, SW2.A, U$7.P$1; no longer C2.1, C3.1, NJM2391.VI, NJM7805.VI
Changed lines of the file:
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@@
 <setting verticaltext="up"/>
 </settings>
-<grid distance="0.1" unitdist="inch" unit="inch" style="lines" multiple="1" display="no" altdistance="0.01" altunitdist="inch" altunit="inch"/>
+<grid distance="50" unitdist="mil" unit="mil" style="lines" multiple="1" display="no" altdistance="0.01" altunitdist="inch" altunit="inch"/>
 <layers>
 <layer number="1" name="Top" color="4" fill="1" visible="no" active="no"/>
@@
 <part name="P+1" library="supply1" library_urn="urn:adsk.eagle:library:371" deviceset="+5V" device=""/>
 <part name="GND1" library="supply1" library_urn="urn:adsk.eagle:library:371" deviceset="GND" device=""/>
-<part name="VDD1" library="supply1" library_urn="urn:adsk.eagle:library:371" deviceset="VDD" device=""/>
 <part name="C1" library="rcl" library_urn="urn:adsk.eagle:library:334" deviceset="C-EU" device="C1608" package3d_urn="urn:adsk.eagle:package:23621/2" value="10uF"/>
 <part name="C2" library="rcl" library_urn="urn:adsk.eagle:library:334" deviceset="C-EU" device="C1608" package3d_urn="urn:adsk.eagle:package:23621/2" value="0.1uF"/>
@@
 <part name="GND6" library="supply1" library_urn="urn:adsk.eagle:library:371" deviceset="GND" device=""/>
 <part name="C6" library="rcl" library_urn="urn:adsk.eagle:library:334" deviceset="C-EU" device="C1608" package3d_urn="urn:adsk.eagle:package:23621/2" value="10uF"/>
+<part name="C8" library="rcl" deviceset="CPOL-US" device="E2.5-6" value="100u"/>
+<part name="VDD5" library="supply1" deviceset="VDD" device=""/>
+<part name="GND7" library="supply1" deviceset="GND" device=""/>
+<part name="U$5" library="Mount_pad" deviceset="2.0" device=""/>
+<part name="U$7" library="Mount_pad" deviceset="2.0" device=""/>
+<part name="GND18" library="supply1" deviceset="GND" device=""/>
+<part name="P+2" library="supply1" library_urn="urn:adsk.eagle:library:371" deviceset="VCC" device=""/>
+<part name="SW2" library="Seeed-OPL-Button" deviceset="DIP-TOGGLE-SWITCH-ON-ON(3+2P-8.8X4.6MM)" device="" value="SK-12D01"/>
 </parts>
 <sheets>
@@
 <instance part="P+1" gate="1" x="7.62" y="58.42" rot="R270"/>
 <instance part="GND1" gate="1" x="-22.86" y="81.28"/>
-<instance part="VDD1" gate="G$1" x="-55.88" y="104.14" rot="R90"/>
 <instance part="C1" gate="G$1" x="-5.08" y="93.98"/>
 <instance part="C2" gate="G$1" x="-40.64" y="93.98"/>
@@
 <instance part="GND6" gate="1" x="149.86" y="129.54" rot="R180"/>
 <instance part="C6" gate="G$1" x="124.46" y="111.76"/>
+<instance part="C8" gate="G$1" x="-78.74" y="97.79"/>
+<instance part="VDD5" gate="G$1" x="-78.74" y="115.57"/>
+<instance part="GND7" gate="1" x="-86.36" y="88.9"/>
+<instance part="U$5" gate="G$1" x="-104.14" y="114.3"/>
+<instance part="U$7" gate="G$1" x="-95.25" y="114.3"/>
+<instance part="GND18" gate="1" x="-78.74" y="88.9"/>
+<instance part="P+2" gate="VCC" x="-50.8" y="114.3"/>
+<instance part="SW2" gate="G$1" x="-64.77" y="118.11" rot="R90"/>
 </instances>
 <busses>
@@
 <net name="VDD" class="0">
 <segment>
-<pinref part="VDD1" gate="G$1" pin="VDD"/>
-<wire x1="-53.34" y1="104.14" x2="-50.8" y2="104.14" width="0.1524" layer="91"/>
-<pinref part="C2" gate="G$1" pin="1"/>
-<wire x1="-50.8" y1="104.14" x2="-40.64" y2="104.14" width="0.1524" layer="91"/>
-<wire x1="-40.64" y1="104.14" x2="-33.02" y2="104.14" width="0.1524" layer="91"/>
-<wire x1="-40.64" y1="96.52" x2="-40.64" y2="104.14" width="0.1524" layer="91"/>
-<junction x="-40.64" y="104.14"/>
-<pinref part="NJM2391" gate="A1" pin="VI"/>
-<junction x="-50.8" y="104.14"/>
-<pinref part="NJM7805" gate="A1" pin="VI"/>
-<wire x1="-50.8" y1="104.14" x2="-50.8" y2="58.42" width="0.1524" layer="91"/>
-<wire x1="-50.8" y1="58.42" x2="-38.1" y2="58.42" width="0.1524" layer="91"/>
-<pinref part="C3" gate="G$1" pin="1"/>
-<wire x1="-38.1" y1="58.42" x2="-30.48" y2="58.42" width="0.1524" layer="91"/>
-<wire x1="-38.1" y1="50.8" x2="-38.1" y2="58.42" width="0.1524" layer="91"/>
-<junction x="-38.1" y="58.42"/>
+<pinref part="C8" gate="G$1" pin="+"/>
+<wire x1="-95.25" y1="104.14" x2="-78.74" y2="104.14" width="0.1524" layer="91"/>
+<pinref part="VDD5" gate="G$1" pin="VDD"/>
+<wire x1="-78.74" y1="104.14" x2="-78.74" y2="113.03" width="0.1524" layer="91"/>
+<junction x="-78.74" y="104.14"/>
+<pinref part="U$7" gate="G$1" pin="P$1"/>
+<wire x1="-78.74" y1="104.14" x2="-67.31" y2="104.14" width="0.1524" layer="91"/>
+<wire x1="-95.25" y1="104.14" x2="-95.25" y2="109.22" width="0.1524" layer="91"/>
+<wire x1="-78.74" y1="100.33" x2="-78.74" y2="104.14" width="0.1524" layer="91"/>
+<junction x="-78.74" y="104.14"/>
+<pinref part="SW2" gate="G$1" pin="A"/>
+<wire x1="-67.31" y1="109.22" x2="-67.31" y2="104.14" width="0.1524" layer="91"/>
 </segment>
 </net>
@@
 <wire x1="132.08" y1="114.3" x2="132.08" y2="109.22" width="0.1524" layer="91"/>
 </segment>
+<segment>
+<pinref part="GND18" gate="1" pin="GND"/>
+<pinref part="C8" gate="G$1" pin="-"/>
+<wire x1="-78.74" y1="92.71" x2="-78.74" y2="91.44" width="0.1524" layer="91"/>
+</segment>
+<segment>
+<wire x1="-86.36" y1="100.33" x2="-86.36" y2="91.44" width="0.1524" layer="91"/>
+<pinref part="GND7" gate="1" pin="GND"/>
+<pinref part="U$5" gate="G$1" pin="P$1"/>
+<wire x1="-86.36" y1="100.33" x2="-104.14" y2="100.33" width="0.1524" layer="91"/>
+<wire x1="-104.14" y1="100.33" x2="-104.14" y2="109.22" width="0.1524" layer="91"/>
+</segment>
 </net>
 <net name="+3V3" class="0">
@@
 </segment>
 </net>
+<net name="VCC" class="0">
+<segment>
+<wire x1="-50.8" y1="111.76" x2="-50.8" y2="104.14" width="0.1524" layer="91"/>
+<pinref part="C2" gate="G$1" pin="1"/>
+<wire x1="-50.8" y1="104.14" x2="-40.64" y2="104.14" width="0.1524" layer="91"/>
+<wire x1="-40.64" y1="104.14" x2="-33.02" y2="104.14" width="0.1524" layer="91"/>
+<wire x1="-40.64" y1="96.52" x2="-40.64" y2="104.14" width="0.1524" layer="91"/>
+<junction x="-40.64" y="104.14"/>
+<pinref part="NJM2391" gate="A1" pin="VI"/>
+<junction x="-50.8" y="104.14"/>
+<pinref part="NJM7805" gate="A1" pin="VI"/>
+<wire x1="-50.8" y1="104.14" x2="-50.8" y2="58.42" width="0.1524" layer="91"/>
+<wire x1="-50.8" y1="58.42" x2="-38.1" y2="58.42" width="0.1524" layer="91"/>
+<pinref part="C3" gate="G$1" pin="1"/>
+<wire x1="-38.1" y1="58.42" x2="-30.48" y2="58.42" width="0.1524" layer="91"/>
+<wire x1="-38.1" y1="50.8" x2="-38.1" y2="58.42" width="0.1524" layer="91"/>
+<junction x="-38.1" y="58.42"/>
+<pinref part="P+2" gate="VCC" pin="VCC"/>
+<pinref part="SW2" gate="G$1" pin="COM"/>
+<wire x1="-64.77" y1="109.22" x2="-64.77" y2="104.14" width="0.1524" layer="91"/>
+<wire x1="-64.77" y1="104.14" x2="-50.8" y2="104.14" width="0.1524" layer="91"/>
+</segment>
+</net>

Commit message: chematic v1.0
Parts:
- removed NJM2391: 7806DT, linear:7806DT
- removed U1: ESP-WROOM-32, esp32 (2):ESP-WROOM-32
- added C10, C9: 0.1u, rcl:C-EUC1608
- added C11, C12, C13: 0.1uF, rcl:C-EUC1608
- added GY-530C, GY-530L, GY-530R: (no value), pinhead:PINHD-1X5M
- added GY-91: (no value), adafruit:PINHD-1X6
- added IC2: LT1963ES8-3.3, linear-technology:LT1963ES8-3.3
- added JP4: (no value), pinhead:PINHD-1X10
- added LED5, LED6, LED7, LED8: WS2812B5050, adafruit:WS2812B5050
- added R2: 10k, rcl:R-EU_R0603
- added R3: 4.7k, rcl:R-EU_R0603
- added R4: 4.7K, rcl:R-EU_R0603
- added SJ1: (no value), SparkFun:SOLDERJUMPER_2WAYS
- added T0, T1, T2, T3, T5, T7: (no value), wirepad:SMD5
- added U$6: PB04, Buzzer:PB04
- added U2: ESP-WROOM-32_NOFLASH, esp32 _my:ESP-WROOM-32_NOFLASH
- C2, C3: value 0.1uF -> 10uF
Connections:
- new net ENCL_A: ML.3, U2.IO34
- new net ENCL_B: ML.4, U2.IO35
- new net ENCR_A: MR.3, U2.SENSOR_VP
- new net ENCR_B: MR.4, U2.SENSOR_VN
- new net I2C_SCL: GY-530C.3, GY-530L.3, GY-530R.3, GY-91.3, JP4.4, R3.1, U2.IO22
- new net I2C_SDA: GY-530C.4, GY-530L.4, GY-530R.4, GY-91.4, JP4.5, R4.1, U2.IO21
- new net IO12: JP4.9, T5.P, U2.IO12
- new net IO15: JP4.8, T3.P, U2.IO15
- new net IO2: JP4.6, T2.P, U2.IO2
- new net IO27: JP4.10, T7.P, U2.IO27
- new net IO4: T0.P, U2.IO4
- new net IO5: JP4.7, U2.IO5
- new net ML_IN1: IC1.AIN1, U2.IO16
- new net ML_IN2: IC1.AIN2, U2.IO17
- new net ML_PWM: IC1.PWMA, U2.IO26
- new net MR_IN1: IC1.BIN1, U2.IO18
- new net MR_IN2: IC1.BIN2, U2.IO19
- new net MR_PWM: IC1.PWMB, U2.IO25
- new net N$10: IC1.AO1, IC1.AO1', ML.1
- new net N$11: IC1.AO2, IC1.AO2', ML.6
- new net N$12: IC1.BO2, IC1.BO2', MR.6
- new net N$13: IC1.BO1, IC1.BO1', MR.1
- new net N$15: LED7.DO, LED8.DI
- new net N$18: LED5.DI, U2.IO13
- new net N$19: GY-530R.5, U2.IO33
- new net N$2: IC2G$1.IN
- new net N$3: GY-530L.5, U2.IO32
- new net N$4: GY-91.6, SJ1.2
- new net N$5: GY-530C.5, U2.IO23
- new net N$6: LED5.DO, LED6.DI
- new net N$7: IC1.STBY, R2.1
- new net N$8: U$6.1, U2.IO14
- new net N$9: LED6.DO, LED7.DI
- net +3V3: now also C9.1, GY-530C.1, GY-530L.1, GY-530R.1, GY-91.1, GY-91.5, IC1.VCC, IC2G$1.OUT, IC2G$1.SENSE, JP4.3, ML.2, MR.2, R2.2, R4.2, SJ1.3, U2.3V3; no longer NJM2391.VO, U1.3V3
- net +5V: now also C11.1, C12.1, C13.1, JP4.2, LED5.VDD, LED6.VDD, LED7.VDD, LED8.VDD
- net EN: now also U2.EN; no longer U1.EN
- net GND: now also C10.2, C11.2, C12.2, C13.2, C9.2, GY-530C.2, GY-530L.2, GY-530R.2, GY-91.2, IC1.GND, IC1.PGND1, IC1.PGND1', IC1.PGND2, IC1.PGND2', IC2G$1.GND, JP4.1, LED5.GND, LED6.GND, LED7.GND, LED8.GND, ML.5, MR.5, SJ1.1, U$6.2, U2.GND@1, U2.GND@2, U2.GND@3, U2.GND@4; no longer NJM2391.GND, U1.GND@1, U1.GND@2, U1.GND@3, U1.GND@4
- net IO0: now also T1.P, U2.IO0; no longer U1.IO0
- net RX: now also U2.RXD0; no longer U1.RXD0
- net TX: now also U2.TXD0; no longer U1.TXD0
- net VCC: now also IC2G$1.!SHDN; no longer NJM2391.VI
- net VDD: now also C10.1, IC1.VM1, IC1.VM2, IC1.VM3
Other:
- note added: "3V3"
- note added: "5V"
- note added: "AD0"
- note added: "BUZ1"
- note added: "ENC_3V3"
- note added: "ENC_A"
- note added: "ENC_B"
- note added: "ENC_GND"
- note added: "GND"
- note added: "I2C_SCL"
- note added: "I2C_SDA"
- note added: "IO12"
- note added: "IO15"
- note added: "IO2"
- note added: "IO27"
- note added: "IO5"
- note added: "M+"
- note added: "M-"
- note added: "NCS"
- note added: "SCL"
- note added: "SDA"
- note added: "VIN"
- note added: "XSHUT"
- moved on the sheet: C6, EN(RESET), IC1, IO0（BOOT), ML, MR

Commit message: board test
Parts:
- renumbered JP1 to SERIAL, JP4 to UNIV
Changed lines of the file:
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@@
 <setting verticaltext="up"/>
 </settings>
-<grid distance="0.1" unitdist="inch" unit="inch" style="lines" multiple="1" display="yes" altdistance="50" altunitdist="mil" altunit="mil"/>
+<grid distance="0.1" unitdist="inch" unit="inch" style="lines" multiple="1" display="no" altdistance="0.01" altunitdist="inch" altunit="inch"/>
 <layers>
 <layer number="1" name="Top" color="4" fill="1" visible="no" active="no"/>
@@
 <parts>
 <part name="IC1" library="adafruit" deviceset="TB6612FNG" device=""/>
-<part name="JP1" library="adafruit" deviceset="PINHD-1X6" device=""/>
+<part name="SERIAL" library="adafruit" deviceset="PINHD-1X6" device=""/>
 <part name="+3V1" library="supply1" library_urn="urn:adsk.eagle:library:371" deviceset="+3V3" device=""/>
 <part name="P+1" library="supply1" library_urn="urn:adsk.eagle:library:371" deviceset="+5V" device=""/>
@@
 <part name="T3" library="wirepad" library_urn="urn:adsk.eagle:library:412" deviceset="SMD5" device="" package3d_urn="urn:adsk.eagle:package:30841/1"/>
 <part name="T7" library="wirepad" library_urn="urn:adsk.eagle:library:412" deviceset="SMD5" device="" package3d_urn="urn:adsk.eagle:package:30841/1"/>
-<part name="JP4" library="pinhead" deviceset="PINHD-1X10" device=""/>
+<part name="UNIV" library="pinhead" deviceset="PINHD-1X10" device=""/>
 <part name="P+4" library="supply1" library_urn="urn:adsk.eagle:library:371" deviceset="+5V" device=""/>
 <part name="GND14" library="supply1" library_urn="urn:adsk.eagle:library:371" deviceset="GND" device=""/>
@@
 <instances>
 <instance part="IC1" gate="G$1" x="-22.86" y="-134.62" rot="R180"/>
-<instance part="JP1" gate="A" x="-48.26" y="-40.64" rot="R180"/>
+<instance part="SERIAL" gate="A" x="-48.26" y="-40.64" rot="R180"/>
 <instance part="+3V1" gate="G$1" x="7.62" y="104.14" rot="R270"/>
 <instance part="P+1" gate="1" x="7.62" y="58.42" rot="R270"/>
@@
 <instance part="T3" gate="1" x="203.2" y="68.58" rot="R180"/>
 <instance part="T7" gate="1" x="137.16" y="81.28"/>
-<instance part="JP4" gate="A" x="182.88" y="-66.04"/>
+<instance part="UNIV" gate="A" x="182.88" y="-66.04"/>
 <instance part="P+4" gate="1" x="165.1" y="-45.72"/>
 <instance part="GND14" gate="1" x="172.72" y="-48.26" rot="R180"/>
@@
 </segment>
 <segment>
-<pinref part="JP1" gate="A" pin="1"/>
+<pinref part="SERIAL" gate="A" pin="1"/>
 <wire x1="-45.72" y1="-48.26" x2="-30.48" y2="-48.26" width="0.1524" layer="91"/>
 <wire x1="-30.48" y1="-48.26" x2="-30.48" y2="-53.34" width="0.1524" layer="91"/>
@@
 </segment>
 <segment>
-<pinref part="JP4" gate="A" pin="1"/>
+<pinref part="UNIV" gate="A" pin="1"/>
 <wire x1="180.34" y1="-55.88" x2="172.72" y2="-55.88" width="0.1524" layer="91"/>
 <wire x1="172.72" y1="-55.88" x2="172.72" y2="-50.8" width="0.1524" layer="91"/>
@@
 </segment>
 <segment>
-<pinref part="JP1" gate="A" pin="3"/>
+<pinref part="SERIAL" gate="A" pin="3"/>
 <pinref part="+3V3" gate="G$1" pin="+3V3"/>
 <wire x1="-45.72" y1="-43.18" x2="-30.48" y2="-43.18" width="0.1524" layer="91"/>
@@
 </segment>
 <segment>
-<pinref part="JP4" gate="A" pin="3"/>
+<pinref part="UNIV" gate="A" pin="3"/>
 <wire x1="180.34" y1="-60.96" x2="160.02" y2="-60.96" width="0.1524" layer="91"/>
 <pinref part="+3V8" gate="G$1" pin="+3V3"/>
@@
 </segment>
 <segment>
-<pinref part="JP4" gate="A" pin="2"/>
+<pinref part="UNIV" gate="A" pin="2"/>
 <wire x1="165.1" y1="-58.42" x2="180.34" y2="-58.42" width="0.1524" layer="91"/>
 <pinref part="P+4" gate="1" pin="+5V"/>
@@
 <pinref part="NDS9936" gate="B" pin="S"/>
 <wire x1="-5.08" y1="-45.72" x2="-5.08" y2="-48.26" width="0.1524" layer="91"/>
-<pinref part="JP1" gate="A" pin="6"/>
+<pinref part="SERIAL" gate="A" pin="6"/>
 <label x="-38.1" y="-35.56" size="1.778" layer="95"/>
 </segment>
@@
 </segment>
 <segment>
-<pinref part="JP1" gate="A" pin="5"/>
+<pinref part="SERIAL" gate="A" pin="5"/>
 <wire x1="-45.72" y1="-38.1" x2="-38.1" y2="-38.1" width="0.1524" layer="91"/>
 <label x="-38.1" y="-38.1" size="1.778" layer="95"/>
@@
 </segment>
 <segment>
-<pinref part="JP1" gate="A" pin="4"/>
+<pinref part="SERIAL" gate="A" pin="4"/>
 <wire x1="-45.72" y1="-40.64" x2="-38.1" y2="-40.64" width="0.1524" layer="91"/>
 <label x="-38.1" y="-40.64" size="1.778" layer="95"/>
@@
 <net name="RTS" class="0">
 <segment>
-<pinref part="JP1" gate="A" pin="2"/>
+<pinref part="SERIAL" gate="A" pin="2"/>
 <pinref part="NDS9936" gate="B" pin="G"/>
 <wire x1="-10.16" y1="-50.8" x2="-15.24" y2="-50.8" width="0.1524" layer="91"/>
@@
 </segment>
 <segment>
-<pinref part="JP4" gate="A" pin="9"/>
+<pinref part="UNIV" gate="A" pin="9"/>
 <wire x1="180.34" y1="-76.2" x2="167.64" y2="-76.2" width="0.1524" layer="91"/>
 <label x="165.1" y="-76.2" size="1.778" layer="95"/>
@@
 </segment>
 <segment>
-<pinref part="JP4" gate="A" pin="4"/>
+<pinref part="UNIV" gate="A" pin="4"/>
 <wire x1="180.34" y1="-63.5" x2="167.64" y2="-63.5" width="0.1524" layer="91"/>
 <label x="165.1" y="-63.5" size="1.778" layer="95"/>
@@
 </segment>
 <segment>
-<pinref part="JP4" gate="A" pin="5"/>
+<pinref part="UNIV" gate="A" pin="5"/>
 <wire x1="167.64" y1="-66.04" x2="180.34" y2="-66.04" width="0.1524" layer="91"/>
 <label x="165.1" y="-66.04" size="1.778" layer="95"/>
@@
 </segment>
 <segment>
-<pinref part="JP4" gate="A" pin="7"/>
+<pinref part="UNIV" gate="A" pin="7"/>
 <wire x1="167.64" y1="-71.12" x2="180.34" y2="-71.12" width="0.1524" layer="91"/>
 <label x="165.1" y="-71.12" size="1.778" layer="95"/>
@@
 </segment>
 <segment>
-<pinref part="JP4" gate="A" pin="6"/>
+<pinref part="UNIV" gate="A" pin="6"/>
 <wire x1="180.34" y1="-68.58" x2="167.64" y2="-68.58" width="0.1524" layer="91"/>
 <label x="165.1" y="-68.58" size="1.778" layer="95"/>
@@
 </segment>
 <segment>
-<pinref part="JP4" gate="A" pin="8"/>
+<pinref part="UNIV" gate="A" pin="8"/>
 <wire x1="180.34" y1="-73.66" x2="167.64" y2="-73.66" width="0.1524" layer="91"/>
 <label x="165.1" y="-73.66" size="1.778" layer="95"/>
@@
 </segment>
 <segment>
-<pinref part="JP4" gate="A" pin="10"/>
+<pinref part="UNIV" gate="A" pin="10"/>
 <wire x1="180.34" y1="-78.74" x2="167.64" y2="-78.74" width="0.1524" layer="91"/>
 <label x="165.1" y="-78.74" size="1.778" layer="95"/>

Commit message: sche fix,board test
Parts:
- removed T7: (no value), wirepad:SMD5
- removed U$6: PB04, Buzzer:PB04
- added BUZ+, BUZ-: (no value), wirepad:SMD2
- added R5: 10k, rcl:R-EU_R0603
- added R6: 20k, rcl:R-EU_R0603
- 5VOUT: device jst-xh:S2B-XH-A -> jst-xh:B2B-XH-A
- UNIV: device pinhead:PINHD-1X10 -> adafruit:PINHD-1X9
Connections:
- net +5V: now also 5VOUT.1; no longer 5VOUT.2
- net GND: now also 5VOUT.2, BUZ-.P, R5.1; no longer 5VOUT.1, U$6.2
- net IO27: now also R5.2, R6.1; no longer T7.P, UNIV.10
- net N$8: now also BUZ+.P; no longer U$6.1
- net VDD: now also R6.2
Other:
- note removed: "BUZ1"
- note removed: "IO27"
- moved on the sheet: 5VOUT, EN(RESET)

Commit message: pdf add
Parts:
- added C14: 0.1uF, rcl:C-EUC1608
Connections:
- net +5V: now also C14.1
- net GND: now also C14.2
Other:
- moved on the sheet: C10, C9, IC1, ML, MR, NDS9936A, NDS9936B, R2, SERIAL, UNIV

Commit message: from office
Parts:
- 5VOUT: device jst-xh:B2B-XH-A -> pinhead:PINHD-1X2
Changed lines of the file:
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@@
 </variantdefs>
 <classes>
-<class number="0" name="default" width="0" drill="0">
+<class number="0" name="default" width="0.4064" drill="0">
+</class>
+<class number="1" name="L" width="1.016" drill="0">
 </class>
 </classes>
@@
 <part name="R6" library="rcl" library_urn="urn:adsk.eagle:library:334" deviceset="R-EU_" device="R0603" package3d_urn="urn:adsk.eagle:package:23555/2" value="20k"/>
 <part name="UNIV" library="adafruit" deviceset="PINHD-1X9" device=""/>
-<part name="5VOUT" library="jst-xh" deviceset="B2B-XH-A" device=""/>
 <part name="BUZ+" library="wirepad" library_urn="urn:adsk.eagle:library:412" deviceset="SMD2" device="" package3d_urn="urn:adsk.eagle:package:30839/1"/>
 <part name="BUZ-" library="wirepad" library_urn="urn:adsk.eagle:library:412" deviceset="SMD2" device="" package3d_urn="urn:adsk.eagle:package:30839/1"/>
 <part name="C14" library="rcl" library_urn="urn:adsk.eagle:library:334" deviceset="C-EU" device="C1608" package3d_urn="urn:adsk.eagle:package:23621/2" value="0.1uF"/>
+<part name="5VOUT" library="pinhead" library_urn="urn:adsk.eagle:library:325" deviceset="PINHD-1X2" device="" package3d_urn="urn:adsk.eagle:package:22435/2"/>
 </parts>
 <sheets>
@@
 <instance part="R6" gate="G$1" x="60.96" y="88.9" rot="R90"/>
 <instance part="UNIV" gate="G$1" x="50.8" y="-10.16"/>
-<instance part="5VOUT" gate="G$1" x="25.4" y="50.8"/>
 <instance part="BUZ+" gate="1" x="142.24" y="58.42"/>
 <instance part="BUZ-" gate="1" x="142.24" y="53.34"/>
 <instance part="C14" gate="G$1" x="231.14" y="17.78"/>
+<instance part="5VOUT" gate="G$1" x="27.94" y="48.26"/>
 </instances>
 <busses>
 </busses>
 <nets>
-<net name="VDD" class="0">
+<net name="VDD" class="1">
 <segment>
 <pinref part="C8" gate="G$1" pin="+"/>
@@
 </segment>
 </net>
-<net name="GND" class="0">
+<net name="GND" class="1">
 <segment>
 <pinref part="GND1" gate="1" pin="GND"/>
@@
 </segment>
 </net>
-<net name="+3V3" class="0">
+<net name="+3V3" class="1">
 <segment>
 <pinref part="C1" gate="G$1" pin="1"/>
@@
 </segment>
 </net>
-<net name="+5V" class="0">
+<net name="+5V" class="1">
 <segment>
 <pinref part="NJM7805" gate="A1" pin="VO"/>
@@
 </segment>
 </net>
-<net name="VCC" class="0">
+<net name="VCC" class="1">
 <segment>
 <wire x1="-50.8" y1="111.76" x2="-50.8" y2="104.14" width="0.1524" layer="91"/>

Commit message: daily
Parts:
- GY-530C, GY-530L, GY-530R: device pinhead:PINHD-1X5M -> pinhead:PINHD-1X5
- renumbered LED5 to LED_FL, LED6 to LED_RL, LED7 to LED_RR, LED8 to LED_FR, U2 to U1
Connections:
- net N$10 renamed ML+
- net N$11 renamed ML-
- net N$12 renamed MR-
- net N$13 renamed MR+
- removed net N$2: IC2G$1.IN
- net +3V3: now also R3.2
- net GND: no longer U1.GND@4
- net N$19: now also GY-530L.5; no longer GY-530R.5
- net N$3: now also GY-530C.5; no longer GY-530L.5
- net N$5: now also GY-530R.5; no longer GY-530C.5
- net VCC: now also IC2G$1.IN
Other:
- moved on the sheet: GY-530C, GY-530L, GY-530R
