File: esp_car.sch (EAGLE design)
At the start: 50 parts, among them IC2 LT1963ES8-3.3, SW2 SK-12D01

Commit message: 電源用MOSFET追加、VDD見直し
Parts:
- added DMG3415U: BSS84, transistor-small-signal:BSS84
- added R7: 100k, rcl:R-EU_R0603
Connections:
- new net N$39: DMG3415U.G, R7.1, SW2.A
- net GND: now also SW2.COM
- net VCC: now also DMG3415U.D; no longer SW2.COM
- net VDD: now also DMG3415U.S, R7.2; no longer SW2.A
Other:
- moved on the sheet: C8, SW2
Changed lines of the file:
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@@
 <?xml version="1.0" encoding="utf-8"?>
 <!DOCTYPE eagle SYSTEM "eagle.dtd">
-<eagle version="9.0.0">
+<eagle version="9.0.1">
 <drawing>
 <settings>
@@
 <part name="TA4805S" library="linear" library_urn="urn:adsk.eagle:library:262" deviceset="78*" device="TV" package3d_urn="urn:adsk.eagle:package:16417/1" technology="8"/>
 <part name="C4" library="rcl" library_urn="urn:adsk.eagle:library:334" deviceset="C-EU" device="C3225" package3d_urn="urn:adsk.eagle:package:23655/2" value="33u"/>
+<part name="DMG3415U" library="transistor-small-signal" library_urn="urn:adsk.eagle:library:401" deviceset="BSS84" device="" package3d_urn="urn:adsk.eagle:package:29752/1"/>
+<part name="R7" library="rcl" library_urn="urn:adsk.eagle:library:334" deviceset="R-EU_" device="R0603" package3d_urn="urn:adsk.eagle:package:23555/2" value="100k"/>
+<part name="GND16" library="supply1" library_urn="urn:adsk.eagle:library:371" deviceset="GND" device=""/>
 </parts>
 <sheets>
@@
 <instance part="GND6" gate="1" x="170.18" y="119.38" rot="R180"/>
 <instance part="C6" gate="G$1" x="146.05" y="111.76"/>
-<instance part="C8" gate="G$1" x="-78.74" y="97.79"/>
-<instance part="VDD5" gate="G$1" x="-78.74" y="114.3"/>
-<instance part="GND7" gate="1" x="-86.36" y="88.9"/>
-<instance part="U$5" gate="G$1" x="-104.14" y="114.3"/>
-<instance part="U$7" gate="G$1" x="-95.25" y="114.3"/>
-<instance part="GND18" gate="1" x="-78.74" y="88.9"/>
+<instance part="C8" gate="G$1" x="-104.14" y="97.79"/>
+<instance part="VDD5" gate="G$1" x="-104.14" y="114.3"/>
+<instance part="GND7" gate="1" x="-111.76" y="88.9"/>
+<instance part="U$5" gate="G$1" x="-129.54" y="114.3"/>
+<instance part="U$7" gate="G$1" x="-120.65" y="114.3"/>
+<instance part="GND18" gate="1" x="-104.14" y="88.9"/>
 <instance part="P+2" gate="VCC" x="-50.8" y="114.3"/>
-<instance part="SW2" gate="G$1" x="-64.77" y="118.11" rot="R90"/>
+<instance part="SW2" gate="G$1" x="-80.01" y="68.58"/>
 <instance part="+3V4" gate="G$1" x="363.22" y="93.98"/>
 <instance part="GND8" gate="1" x="358.14" y="11.43"/>
@@
 <attribute name="VALUE" x="-3.556" y="43.561" size="1.778" layer="96"/>
 </instance>
+<instance part="DMG3415U" gate="G$1" x="-78.74" y="104.14" rot="R90"/>
+<instance part="R7" gate="G$1" x="-91.44" y="93.98" rot="R90"/>
+<instance part="GND16" gate="1" x="-91.44" y="55.88"/>
 </instances>
 <busses>
@@
 <segment>
 <pinref part="C8" gate="G$1" pin="+"/>
-<wire x1="-95.25" y1="104.14" x2="-78.74" y2="104.14" width="0.1524" layer="91"/>
+<wire x1="-120.65" y1="104.14" x2="-104.14" y2="104.14" width="0.1524" layer="91"/>
 <pinref part="VDD5" gate="G$1" pin="VDD"/>
-<wire x1="-78.74" y1="104.14" x2="-78.74" y2="111.76" width="0.1524" layer="91"/>
-<junction x="-78.74" y="104.14"/>
+<wire x1="-104.14" y1="104.14" x2="-104.14" y2="111.76" width="0.1524" layer="91"/>
+<junction x="-104.14" y="104.14"/>
 <pinref part="U$7" gate="G$1" pin="P$1"/>
-<wire x1="-78.74" y1="104.14" x2="-67.31" y2="104.14" width="0.1524" layer="91"/>
-<wire x1="-95.25" y1="104.14" x2="-95.25" y2="109.22" width="0.1524" layer="91"/>
-<wire x1="-78.74" y1="100.33" x2="-78.74" y2="104.14" width="0.1524" layer="91"/>
-<junction x="-78.74" y="104.14"/>
-<pinref part="SW2" gate="G$1" pin="A"/>
-<wire x1="-67.31" y1="109.22" x2="-67.31" y2="104.14" width="0.1524" layer="91"/>
+<wire x1="-104.14" y1="104.14" x2="-91.44" y2="104.14" width="0.1524" layer="91"/>
+<wire x1="-120.65" y1="104.14" x2="-120.65" y2="109.22" width="0.1524" layer="91"/>
+<wire x1="-104.14" y1="100.33" x2="-104.14" y2="104.14" width="0.1524" layer="91"/>
+<junction x="-104.14" y="104.14"/>
+<wire x1="-91.44" y1="104.14" x2="-91.44" y2="99.06" width="0.1524" layer="91"/>
+<pinref part="R7" gate="G$1" pin="2"/>
+<junction x="-91.44" y="104.14"/>
+<pinref part="DMG3415U" gate="G$1" pin="S"/>
+<wire x1="-83.82" y1="104.14" x2="-91.44" y2="104.14" width="0.1524" layer="91"/>
 </segment>
 <segment>
@@
 <pinref part="GND18" gate="1" pin="GND"/>
 <pinref part="C8" gate="G$1" pin="-"/>
-<wire x1="-78.74" y1="92.71" x2="-78.74" y2="91.44" width="0.1524" layer="91"/>
-</segment>
-<segment>
-<wire x1="-86.36" y1="100.33" x2="-86.36" y2="91.44" width="0.1524" layer="91"/>
+<wire x1="-104.14" y1="92.71" x2="-104.14" y2="91.44" width="0.1524" layer="91"/>
+</segment>
+<segment>
+<wire x1="-111.76" y1="100.33" x2="-111.76" y2="91.44" width="0.1524" layer="91"/>
 <pinref part="GND7" gate="1" pin="GND"/>
 <pinref part="U$5" gate="G$1" pin="P$1"/>
-<wire x1="-86.36" y1="100.33" x2="-104.14" y2="100.33" width="0.1524" layer="91"/>
-<wire x1="-104.14" y1="100.33" x2="-104.14" y2="109.22" width="0.1524" layer="91"/>
+<wire x1="-111.76" y1="100.33" x2="-129.54" y2="100.33" width="0.1524" layer="91"/>
+<wire x1="-129.54" y1="100.33" x2="-129.54" y2="109.22" width="0.1524" layer="91"/>
 </segment>
 <segment>
@@
 <wire x1="60.96" y1="68.58" x2="60.96" y2="63.5" width="0.1524" layer="91"/>
 </segment>
+<segment>
+<pinref part="SW2" gate="G$1" pin="COM"/>
+<wire x1="-88.9" y1="68.58" x2="-91.44" y2="68.58" width="0.1524" layer="91"/>
+<wire x1="-91.44" y1="68.58" x2="-91.44" y2="58.42" width="0.1524" layer="91"/>
+<pinref part="GND16" gate="1" pin="GND"/>
+</segment>
 </net>
 <net name="+3V3" class="1">
@@
 <junction x="-38.1" y="58.42"/>
 <pinref part="P+2" gate="VCC" pin="VCC"/>
-<pinref part="SW2" gate="G$1" pin="COM"/>
-<wire x1="-64.77" y1="109.22" x2="-64.77" y2="104.14" width="0.1524" layer="91"/>
-<wire x1="-64.77" y1="104.14" x2="-50.8" y2="104.14" width="0.1524" layer="91"/>
+<wire x1="-73.66" y1="104.14" x2="-50.8" y2="104.14" width="0.1524" layer="91"/>
 <pinref part="IC2" gate="G$1" pin="!SHDN"/>
 <pinref part="IC2" gate="G$1" pin="IN"/>
 <wire x1="-40.64" y1="104.14" x2="-33.02" y2="104.14" width="0.1524" layer="91"/>
 <pinref part="TA4805S" gate="A1" pin="VI"/>
+<pinref part="DMG3415U" gate="G$1" pin="D"/>
 </segment>
 </net>
@@
 </segment>
 </net>
+<net name="N$39" class="0">
+<segment>
+<pinref part="R7" gate="G$1" pin="1"/>
+<wire x1="-91.44" y1="88.9" x2="-91.44" y2="83.82" width="0.1524" layer="91"/>
+<wire x1="-91.44" y1="83.82" x2="-91.44" y2="71.12" width="0.1524" layer="91"/>
+<wire x1="-88.9" y1="71.12" x2="-91.44" y2="71.12" width="0.1524" layer="91"/>
+<pinref part="SW2" gate="G$1" pin="A"/>
+<junction x="-91.44" y="83.82"/>
+<pinref part="DMG3415U" gate="G$1" pin="G"/>
+<wire x1="-91.44" y1="83.82" x2="-81.28" y2="83.82" width="0.1524" layer="91"/>
+<wire x1="-81.28" y1="83.82" x2="-81.28" y2="99.06" width="0.1524" layer="91"/>
+</segment>
+</net>

Commit message: esp32のviaの径設定ミス修正、NMOS向き修正、配線やり直し完了
Parts:
- removed ESP32: ESP-WROOM-32_NOFLASH_PINHEAD, esp32 _my:ESP-WROOM-32_NOFLASH_PINHEAD
- added TB6612: TB6612_NEW, adafruit_my:TB6612_NEW
- U$1: value TB6612_NEW -> ESP-WROOM-32_NOFLASH_PINHEAD; device adafruit_my:TB6612_NEW -> esp32 _my:ESP-WROOM-32_NOFLASH_PINHEAD
- renumbered EN(RESET) to RST, IO0（BOOT) to BOOT, SW2 to SW1
Connections:
- net +3V3: now also TB6612.VCC, U$1.3V3; no longer ESP32.3V3, U$1.VCC
- net EN: now also U$1.EN; no longer ESP32.EN
- net ENCL_A: now also U$1.IO34; no longer ESP32.IO34
- net ENCL_B: now also U$1.IO35; no longer ESP32.IO35
- net ENCR_A: now also U$1.SENSOR_VP; no longer ESP32.SENSOR_VP
- net ENCR_B: now also U$1.SENSOR_VN; no longer ESP32.SENSOR_VN
- net GND: now also TB6612.GND, TB6612.PGND1, TB6612.PGND2, U$1.GND@1, U$1.GND@2, U$1.GND@3; no longer ESP32.GND@1, ESP32.GND@2, ESP32.GND@3, U$1.GND, U$1.PGND1, U$1.PGND2
- net I2C_SCL: now also U$1.IO22; no longer ESP32.IO22
- net I2C_SDA: now also U$1.IO21; no longer ESP32.IO21
- net IO0: now also U$1.IO0; no longer ESP32.IO0
- net IO12: now also U$1.IO12; no longer ESP32.IO12
- net IO15: now also U$1.IO15; no longer ESP32.IO15
- net IO2: now also U$1.IO2; no longer ESP32.IO2
- net IO27: now also U$1.IO27; no longer ESP32.IO27
- net IO4: now also U$1.IO4; no longer ESP32.IO4
- net IO5: now also U$1.IO5; no longer ESP32.IO5
- net ML-: now also TB6612.AO1; no longer U$1.AO1
- net ML_IN1: now also TB6612.AIN1, U$1.IO16; no longer ESP32.IO16, U$1.AIN1
- net ML_IN2: now also TB6612.AIN2, U$1.IO17; no longer ESP32.IO17, U$1.AIN2
- net ML_PWM: now also TB6612.PWMA, U$1.IO26; no longer ESP32.IO26, U$1.PWMA
- net MR+: now also TB6612.BO1; no longer U$1.BO1
- net MR-: now also TB6612.BO2; no longer U$1.BO2
- net MR_IN1: now also TB6612.BIN1, U$1.IO18; no longer ESP32.IO18, U$1.BIN1
- net MR_IN2: now also TB6612.BIN2, U$1.IO19; no longer ESP32.IO19, U$1.BIN2
- net MR_PWM: now also TB6612.PWMB, U$1.IO25; no longer ESP32.IO25, U$1.PWMB
- net N$18: now also U$1.IO13; no longer ESP32.IO13
- net N$19: now also U$1.IO33; no longer ESP32.IO33
- net N$3: now also U$1.IO32; no longer ESP32.IO32
- net N$38: now also TB6612.AO2; no longer U$1.AO2
- net N$5: now also U$1.IO23; no longer ESP32.IO23
- net N$7: now also TB6612.STBY; no longer U$1.STBY
- net N$8: now also U$1.IO14; no longer ESP32.IO14
- net RX: now also U$1.RXD0; no longer ESP32.RXD0
- net TX: now also U$1.TXD0; no longer ESP32.TXD0
- net VDD: now also TB6612.VM1, TB6612.VM2; no longer U$1.VM1, U$1.VM2
