File: circuit/esp_car.brd (EAGLE design)
At the start: 81.6 x 84 mm, 52 parts, among them IC2 LT1963ES8-3.3, SW1 SK-12D01

Commit message: 抵抗値の修正
Parts:
- R6: value 20k -> 22k
Changed lines of the file:
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@@
 <attribute name="SPICEPREFIX" value="R" x="33.4" y="53.8" size="1.778" layer="27" rot="R90" display="off"/>
 </element>
-<element name="R6" library="rcl" library_urn="urn:adsk.eagle:library:334" package="R0603" package3d_urn="urn:adsk.eagle:package:23555/2" value="20k" x="33.4" y="56.8" smashed="yes" rot="R90">
+<element name="R6" library="rcl" library_urn="urn:adsk.eagle:library:334" package="R0603" package3d_urn="urn:adsk.eagle:package:23555/2" value="22k" x="33.4" y="56.8" smashed="yes" rot="R90">
 <attribute name="NAME" x="34.5892" y="59.7906" size="1.27" layer="25" rot="R180"/>
 <attribute name="SPICEPREFIX" value="R" x="33.4" y="56.8" size="1.778" layer="27" rot="R90" display="off"/>
