File: circuit/esp_car.sch (EAGLE design)
At the start: 52 parts, among them IC2 LT1963ES8-3.3, SW1 SK-12D01

Commit message: 抵抗値の修正
Parts:
- R6: value 20k -> 22k
Changed lines of the file:
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@@
 <part name="VDD1" library="supply1" deviceset="VDD" device=""/>
 <part name="R5" library="rcl" library_urn="urn:adsk.eagle:library:334" deviceset="R-EU_" device="R0603" package3d_urn="urn:adsk.eagle:package:23555/2" value="10k"/>
-<part name="R6" library="rcl" library_urn="urn:adsk.eagle:library:334" deviceset="R-EU_" device="R0603" package3d_urn="urn:adsk.eagle:package:23555/2" value="20k"/>
+<part name="R6" library="rcl" library_urn="urn:adsk.eagle:library:334" deviceset="R-EU_" device="R0603" package3d_urn="urn:adsk.eagle:package:23555/2" value="22k"/>
 <part name="UNIV" library="adafruit" deviceset="PINHD-1X9" device=""/>
 <part name="BUZ+" library="wirepad" library_urn="urn:adsk.eagle:library:412" deviceset="SMD2" device="" package3d_urn="urn:adsk.eagle:package:30839/1"/>
